Commit message: changed mesh location for testing

File: mujoco_ros2_pkg/urdf/arm_base_link_xacro.xacro (robot description, xacro)
@@ -5,5 +5,5 @@
             <origin xyz="0.0 0.0 0.0" rpy="0.0 0.0 0.0" />
             <geometry>
-                <mesh filename="package://dofbot_description/meshes/low_poly/dofbot/visual/base_link_low_poly.stl" />
+                <mesh filename="package://mujoco_ros2_pkg/meshes/low_poly/dofbot/visual/base_link_low_poly.stl" />
             </geometry>
             <material name="eerie_black" />
@@ -12,5 +12,5 @@
             <origin xyz="0.0 0.0 0.0" rpy="0.0 0.0 0.0" />
             <geometry>
-                <mesh filename="package://dofbot_description/meshes/low_poly/dofbot/visual/base_link_low_poly.stl" />
+                <mesh filename="package://mujoco_ros2_pkg/meshes/low_poly/dofbot/visual/base_link_low_poly.stl" />
             </geometry>
         </collision>

File: mujoco_ros2_pkg/urdf/dofbot_arm_urdf.xacro (robot description, xacro)
@@ -30,5 +30,5 @@
             <origin xyz="0 0 0" rpy="0 0 0" />
             <geometry>
-                <mesh filename="package://dofbot_description/meshes/low_poly/dofbot/visual/arm_link1_low_poly.stl" />
+                <mesh filename="package://mujoco_ros2_pkg/meshes/low_poly/dofbot/visual/arm_link1_low_poly.stl" />
             </geometry>
             <material name="pigment_green" />
@@ -37,5 +37,5 @@
             <origin xyz="0 0 0" rpy="0 0 0" />
             <geometry>
-                <mesh filename="package://dofbot_description/meshes/low_poly/dofbot/visual/arm_link1_low_poly.stl" />
+                <mesh filename="package://mujoco_ros2_pkg/meshes/low_poly/dofbot/visual/arm_link1_low_poly.stl" />
             </geometry>
         </collision>
@@ -59,5 +59,5 @@
             <origin xyz="0 0 0" rpy="0 0 0" />
             <geometry>
-                <mesh filename="package://dofbot_description/meshes/low_poly/dofbot/visual/arm_link2_low_poly.stl" />
+                <mesh filename="package://mujoco_ros2_pkg/meshes/low_poly/dofbot/visual/arm_link2_low_poly.stl" />
             </geometry>
             <material name="pigment_green" />
@@ -66,5 +66,5 @@
             <origin xyz="0 0 0" rpy="0 0 0" />
             <geometry>
-                <mesh filename="package://dofbot_description/meshes/low_poly/dofbot/visual/arm_link2_low_poly.stl" />
+                <mesh filename="package://mujoco_ros2_pkg/meshes/low_poly/dofbot/visual/arm_link2_low_poly.stl" />
             </geometry>
         </collision>
@@ -88,5 +88,5 @@
             <origin xyz="0 0 0" rpy="0 0 0" />
             <geometry>
-                <mesh filename="package://dofbot_description/meshes/low_poly/dofbot/visual/arm_link3_low_poly.stl" />
+                <mesh filename="package://mujoco_ros2_pkg/meshes/low_poly/dofbot/visual/arm_link3_low_poly.stl" />
             </geometry>
             <material name="pigment_green" />
@@ -95,5 +95,5 @@
             <origin xyz="0 0 0" rpy="0 0 0" />
             <geometry>
-                <mesh filename="package://dofbot_description/meshes/low_poly/dofbot/visual/arm_link3_low_poly.stl" />
+                <mesh filename="package://mujoco_ros2_pkg/meshes/low_poly/dofbot/visual/arm_link3_low_poly.stl" />
             </geometry>
         </collision>
@@ -117,5 +117,5 @@
             <origin xyz="0 0 0" rpy="0 0 0" />
             <geometry>
-                <mesh filename="package://dofbot_description/meshes/low_poly/dofbot/visual/arm_link4_low_poly.stl" />
+                <mesh filename="package://mujoco_ros2_pkg/meshes/low_poly/dofbot/visual/arm_link4_low_poly.stl" />
             </geometry>
             <material name="pigment_green" />
@@ -124,5 +124,5 @@
             <origin xyz="0 0 0" rpy="0 0 0" />
             <geometry>
-                <mesh filename="package://dofbot_description/meshes/low_poly/dofbot/visual/arm_link4_low_poly.stl" />
+                <mesh filename="package://mujoco_ros2_pkg/meshes/low_poly/dofbot/visual/arm_link4_low_poly.stl" />
             </geometry>
         </collision>
@@ -146,5 +146,5 @@
             <origin xyz="0 0 0" rpy="0 0 0" />
             <geometry>
-                <mesh filename="package://dofbot_description/meshes/low_poly/dofbot/visual/arm_link5_low_poly.stl" />
+                <mesh filename="package://mujoco_ros2_pkg/meshes/low_poly/dofbot/visual/arm_link5_low_poly.stl" />
             </geometry>
             <material name="eerie_black" />
@@ -153,5 +153,5 @@
             <origin xyz="0 0 0" rpy="0 0 0" />
             <geometry>
-                <mesh filename="package://dofbot_description/meshes/low_poly/dofbot/visual/arm_link5_low_poly.stl" />
+                <mesh filename="package://mujoco_ros2_pkg/meshes/low_poly/dofbot/visual/arm_link5_low_poly.stl" />
             </geometry>
         </collision>
@@ -176,5 +176,5 @@
             <origin xyz="0 0 0" rpy="0 0 0" />
             <geometry>
-                <mesh filename="package://dofbot_description/meshes/low_poly/dofbot/visual/rgrip_finger1_low_poly.stl" />
+                <mesh filename="package://mujoco_ros2_pkg/meshes/low_poly/dofbot/visual/rgrip_finger1_low_poly.stl" />
             </geometry>
             <material name="yinmn_blue" />
@@ -183,5 +183,5 @@
             <origin xyz="0 0 0" rpy="0 0 0" />
             <geometry>
-                <mesh filename="package://dofbot_description/meshes/low_poly/dofbot/visual/rgrip_finger1_low_poly.stl" />
+                <mesh filename="package://mujoco_ros2_pkg/meshes/low_poly/dofbot/visual/rgrip_finger1_low_poly.stl" />
             </geometry>
         </collision>
@@ -206,5 +206,5 @@
             <origin xyz="0 0 0" rpy="0 0 0" />
             <geometry>
-                <mesh filename="package://dofbot_description/meshes/low_poly/dofbot/visual/rgrip_finger2_low_poly.stl" />
+                <mesh filename="package://mujoco_ros2_pkg/meshes/low_poly/dofbot/visual/rgrip_finger2_low_poly.stl" />
             </geometry>
             <material name="oxford_blue" />
@@ -213,5 +213,5 @@
             <origin xyz="0 0 0" rpy="0 0 0" />
             <geometry>
-                <mesh filename="package://dofbot_description/meshes/low_poly/dofbot/visual/rgrip_finger2_low_poly.stl" />
+                <mesh filename="package://mujoco_ros2_pkg/meshes/low_poly/dofbot/visual/rgrip_finger2_low_poly.stl" />
             </geometry>
         </collision>
@@ -236,5 +236,5 @@
             <origin xyz="0 0 0" rpy="0 0 0" />
             <geometry>
-                <mesh filename="package://dofbot_description/meshes/low_poly/dofbot/visual/rgrip_finger3_low_poly.stl" />
+                <mesh filename="package://mujoco_ros2_pkg/meshes/low_poly/dofbot/visual/rgrip_finger3_low_poly.stl" />
             </geometry>
             <material name="silver_lake_blue" />
@@ -243,5 +243,5 @@
             <origin xyz="0 0 0" rpy="0 0 0" />
             <geometry>
-                <mesh filename="package://dofbot_description/meshes/low_poly/dofbot/visual/rgrip_finger3_low_poly.stl" />
+                <mesh filename="package://mujoco_ros2_pkg/meshes/low_poly/dofbot/visual/rgrip_finger3_low_poly.stl" />
             </geometry>
         </collision>
@@ -266,5 +266,5 @@
             <origin xyz="0 0 0" rpy="0 0 0" />
             <geometry>
-                <mesh filename="package://dofbot_description/meshes/low_poly/dofbot/visual/lgrip_finger1_low_poly.stl" />
+                <mesh filename="package://mujoco_ros2_pkg/meshes/low_poly/dofbot/visual/lgrip_finger1_low_poly.stl" />
             </geometry>
             <material name="yinmn_blue" />
@@ -273,5 +273,5 @@
             <origin xyz="0 0 0" rpy="0 0 0" />
             <geometry>
-                <mesh filename="package://dofbot_description/meshes/low_poly/dofbot/visual/lgrip_finger1_low_poly.stl" />
+                <mesh filename="package://mujoco_ros2_pkg/meshes/low_poly/dofbot/visual/lgrip_finger1_low_poly.stl" />
             </geometry>
         </collision>
@@ -296,5 +296,5 @@
             <origin xyz="0 0 0" rpy="0 0 0" />
             <geometry>
-                <mesh filename="package://dofbot_description/meshes/low_poly/dofbot/visual/lgrip_finger2_low_poly.stl" />
+                <mesh filename="package://mujoco_ros2_pkg/meshes/low_poly/dofbot/visual/lgrip_finger2_low_poly.stl" />
             </geometry>
             <material name="oxford_blue" />
@@ -303,5 +303,5 @@
             <origin xyz="0 0 0" rpy="0 0 0" />
             <geometry>
-                <mesh filename="package://dofbot_description/meshes/low_poly/dofbot/visual/lgrip_finger2_low_poly.stl" />
+                <mesh filename="package://mujoco_ros2_pkg/meshes/low_poly/dofbot/visual/lgrip_finger2_low_poly.stl" />
             </geometry>
         </collision>
@@ -326,5 +326,5 @@
             <origin xyz="0 0 0" rpy="0 0 0" />
             <geometry>
-                <mesh filename="package://dofbot_description/meshes/low_poly/dofbot/visual/lgrip_finger3_low_poly.stl" />
+                <mesh filename="package://mujoco_ros2_pkg/meshes/low_poly/dofbot/visual/lgrip_finger3_low_poly.stl" />
             </geometry>
             <material name="silver_lake_blue" />
@@ -333,5 +333,5 @@
             <origin xyz="0 0 0" rpy="0 0 0" />
             <geometry>
-                <mesh filename="package://dofbot_description/meshes/low_poly/dofbot/visual/lgrip_finger3_low_poly.stl" />
+                <mesh filename="package://mujoco_ros2_pkg/meshes/low_poly/dofbot/visual/lgrip_finger3_low_poly.stl" />
             </geometry>
         </collision>

File: mujoco_ros2_pkg/urdf/dofbot_trajectory_controller.xacro (robot description, xacro)
@@ -3,6 +3,6 @@
     <xacro:property name="package_name" value="mujoco_ros2_pkg"/>
     <xacro:include filename="$(find ${package_name})/urdf/dofbot_arm_urdf.xacro"/>
-    <!--<xacro:include filename="$(find ${package_name})/urdf/dofbot_gz_properties.xacro"/>
-    <xacro:include filename="$(find ${package_name})/urdf/trajectory_controller.xacro"/>-->
+    <!--<xacro:include filename="$(find ${package_name})/urdf/dofbot_gz_properties.xacro"/>-->
+    <xacro:include filename="$(find ${package_name})/urdf/trajectory_controller.xacro"/>
     <xacro:include filename="$(find ${package_name})/urdf/xacro_properties.xacro"/>
     <!--<xacro:include filename="$(find ${package_name})/urdf/monocular_camera_sensor.xacro"/>-->

File: mujoco_ros2_pkg/urdf/monocular_camera_sensor.xacro (robot description, xacro)
@@ -12,5 +12,5 @@
           <origin xyz="0 0 0" rpy="0 0 0"/>
           <geometry>
-              <mesh filename="package://dofbot_description/meshes/low_poly/sensor/visual/mono_link_low_poly.stl"/>
+              <mesh filename="package://mujoco_ros2_pkg/meshes/low_poly/sensor/visual/mono_link_low_poly.stl"/>
           </geometry>
           <material name="">
@@ -21,5 +21,5 @@
           <origin xyz="0 0 0" rpy="0 0 0"/>
           <geometry>
-              <mesh filename="package://dofbot_description/meshes/low_poly/sensor/visual/mono_link_low_poly.stl"/>
+              <mesh filename="package://mujoco_ros2_pkg/meshes/low_poly/sensor/visual/mono_link_low_poly.stl"/>
           </geometry>
       </collision>

File: mujoco_ros2_pkg/urdf/trajectory_controller.xacro (robot description, xacro)
@@ -2,82 +2,56 @@
 <!--Aqui comienza el robot-->
 <robot name="trajectory_controller" xmlns:xacro="http://ros.org/wiki/xacro" >
-    <ros2_control name="GazeboSystem" type="system">
+    <ros2_control name="MujocoSystem" type="system">
         <hardware>
-            <plugin>gazebo_ros2_control/GazeboSystem</plugin>
+            <plugin>mujoco_ros2_control/MujocoSystem</plugin>
         </hardware>
         <joint name="arm_joint_01">
-            <command_interface name="position"/>
-            <state_interface name="position"/>
+            <command_interface name="position" />
+            <state_interface name="position">
+                <param name="initial_value">1.0</param>
+            </state_interface>
             <state_interface name="velocity"/>
             <state_interface name="effort"/>
         </joint>
         <joint name="arm_joint_02">
-            <command_interface name="position"/>
-            <state_interface name="position"/>
+            <command_interface name="position" />
+            <state_interface name="position">
+                <param name="initial_value">1.0</param>
+            </state_interface>
             <state_interface name="velocity"/>
             <state_interface name="effort"/>
         </joint>
         <joint name="arm_joint_03">
-            <command_interface name="position"/>
-            <state_interface name="position"/>
+            <command_interface name="position" />
+            <state_interface name="position">
+                <param name="initial_value">1.0</param>
+            </state_interface>
             <state_interface name="velocity"/>
             <state_interface name="effort"/>
         </joint>
-        <joint name="arm_joint_04">
-            <command_interface name="position"/>
-            <state_interface name="position"/>
+        <!--<joint name="arm_joint_04">
+            <command_interface name="position" />
+            <state_interface name="position">
+                <param name="initial_value">1.0</param>
+            </state_interface>
             <state_interface name="velocity"/>
             <state_interface name="effort"/>
         </joint>
         <joint name="arm_joint_05">
-            <command_interface name="position"/>
-            <state_interface name="position"/>
+            <command_interface name="position" />
+            <state_interface name="position">
+                <param name="initial_value">1.0</param>
+            </state_interface>
             <state_interface name="velocity"/>
             <state_interface name="effort"/>
-        </joint>
-        <joint name="grip_joint">
-            <command_interface name="position"/>
-            <state_interface name="position"/>
-            <state_interface name="velocity"/>
-            <state_interface name="effort"/>
-        </joint>
-        <joint name="rfinger_joint_01">
-            <command_interface name="position"/>
-            <state_interface name="position"/>
-            <state_interface name="velocity"/>
-            <state_interface name="effort"/>
-        </joint>
-        <joint name="rfinger_joint_02">
-            <command_interface name="position"/>
-            <state_interface name="position"/>
-            <state_interface name="velocity"/>
-            <state_interface name="effort"/>
-        </joint>
-        <joint name="lfinger_grip_joint_01">
-            <command_interface name="position"/>
-            <state_interface name="position"/>
-            <state_interface name="velocity"/>
-            <state_interface name="effort"/>
-        </joint>
-        <joint name="lfinger_grip_joint_02">
-            <command_interface name="position"/>
-            <state_interface name="position"/>
-            <state_interface name="velocity"/>
-            <state_interface name="effort"/>
-        </joint>
-        <joint name="lfinger_grip_joint_03">
-            <command_interface name="position"/>
-            <state_interface name="position"/>
+        </joint>-->
+        <joint name="arm_base_link">
+            <command_interface name="position" />
+            <state_interface name="position">
+                <param name="initial_value">1.0</param>
+            </state_interface>
             <state_interface name="velocity"/>
             <state_interface name="effort"/>
         </joint>
     </ros2_control>
-    <!-- Pluging de control -->
-    <gazebo>
-        <plugin filename="libgazebo_ros2_control.so" name="gazebo_ros2_control" >
-            <robot_param>robot_description</robot_param>
-            <robot_param_node>robot_state_publisher</robot_param_node>
-            <parameters>$(find dofbot_description)/config/dofbot_trajectory_controller.yaml</parameters>
-        </plugin>
-    </gazebo>
 </robot>
