Commit message: add full urdf for mujoco and stl

File: mujoco_ros2_pkg/FullURDF/full_urdf.xacro (robot description, xacro)
@@ -1,5 +1,5 @@
 <?xml version="1.0" ?>
 <!-- =================================================================================== -->
-<!-- |    This document was autogenerated by xacro from ../urdf/dofbot_trajectory_controller.xacro | -->
+<!-- |    This document was autogenerated by xacro from src/mujoco_ros2_pkg/urdf/dofbot_trajectory_controller.xacro | -->
 <!-- |    EDITING THIS FILE BY HAND IS NOT RECOMMENDED                                 | -->
 <!-- =================================================================================== -->
@@ -25,5 +25,5 @@
       <origin rpy="0.0 0.0 0.0" xyz="0.0 0.0 0.0"/>
       <geometry>
-        <mesh filename="package://dofbot_description/meshes/low_poly/dofbot/visual/base_link_low_poly.stl"/>
+        <mesh filename="package://mujoco_ros2_pkg/meshes/low_poly/dofbot/visual/base_link_low_poly.stl"/>
       </geometry>
       <material name="eerie_black"/>
@@ -32,5 +32,5 @@
       <origin rpy="0.0 0.0 0.0" xyz="0.0 0.0 0.0"/>
       <geometry>
-        <mesh filename="package://dofbot_description/meshes/low_poly/dofbot/visual/base_link_low_poly.stl"/>
+        <mesh filename="package://mujoco_ros2_pkg/meshes/low_poly/dofbot/visual/base_link_low_poly.stl"/>
       </geometry>
     </collision>
@@ -51,5 +51,5 @@
       <origin rpy="0 0 0" xyz="0 0 0"/>
       <geometry>
-        <mesh filename="package://dofbot_description/meshes/low_poly/dofbot/visual/arm_link1_low_poly.stl"/>
+        <mesh filename="package://mujoco_ros2_pkg/meshes/low_poly/dofbot/visual/arm_link1_low_poly.stl"/>
       </geometry>
       <material name="pigment_green"/>
@@ -58,5 +58,5 @@
       <origin rpy="0 0 0" xyz="0 0 0"/>
       <geometry>
-        <mesh filename="package://dofbot_description/meshes/low_poly/dofbot/visual/arm_link1_low_poly.stl"/>
+        <mesh filename="package://mujoco_ros2_pkg/meshes/low_poly/dofbot/visual/arm_link1_low_poly.stl"/>
       </geometry>
     </collision>
@@ -80,5 +80,5 @@
       <origin rpy="0 0 0" xyz="0 0 0"/>
       <geometry>
-        <mesh filename="package://dofbot_description/meshes/low_poly/dofbot/visual/arm_link2_low_poly.stl"/>
+        <mesh filename="package://mujoco_ros2_pkg/meshes/low_poly/dofbot/visual/arm_link2_low_poly.stl"/>
       </geometry>
       <material name="pigment_green"/>
@@ -87,5 +87,5 @@
       <origin rpy="0 0 0" xyz="0 0 0"/>
       <geometry>
-        <mesh filename="package://dofbot_description/meshes/low_poly/dofbot/visual/arm_link2_low_poly.stl"/>
+        <mesh filename="package://mujoco_ros2_pkg/meshes/low_poly/dofbot/visual/arm_link2_low_poly.stl"/>
       </geometry>
     </collision>
@@ -109,5 +109,5 @@
       <origin rpy="0 0 0" xyz="0 0 0"/>
       <geometry>
-        <mesh filename="package://dofbot_description/meshes/low_poly/dofbot/visual/arm_link3_low_poly.stl"/>
+        <mesh filename="package://mujoco_ros2_pkg/meshes/low_poly/dofbot/visual/arm_link3_low_poly.stl"/>
       </geometry>
       <material name="pigment_green"/>
@@ -116,5 +116,5 @@
       <origin rpy="0 0 0" xyz="0 0 0"/>
       <geometry>
-        <mesh filename="package://dofbot_description/meshes/low_poly/dofbot/visual/arm_link3_low_poly.stl"/>
+        <mesh filename="package://mujoco_ros2_pkg/meshes/low_poly/dofbot/visual/arm_link3_low_poly.stl"/>
       </geometry>
     </collision>
@@ -138,5 +138,5 @@
       <origin rpy="0 0 0" xyz="0 0 0"/>
       <geometry>
-        <mesh filename="package://dofbot_description/meshes/low_poly/dofbot/visual/arm_link4_low_poly.stl"/>
+        <mesh filename="package://mujoco_ros2_pkg/meshes/low_poly/dofbot/visual/arm_link4_low_poly.stl"/>
       </geometry>
       <material name="pigment_green"/>
@@ -145,5 +145,5 @@
       <origin rpy="0 0 0" xyz="0 0 0"/>
       <geometry>
-        <mesh filename="package://dofbot_description/meshes/low_poly/dofbot/visual/arm_link4_low_poly.stl"/>
+        <mesh filename="package://mujoco_ros2_pkg/meshes/low_poly/dofbot/visual/arm_link4_low_poly.stl"/>
       </geometry>
     </collision>
@@ -167,5 +167,5 @@
       <origin rpy="0 0 0" xyz="0 0 0"/>
       <geometry>
-        <mesh filename="package://dofbot_description/meshes/low_poly/dofbot/visual/arm_link5_low_poly.stl"/>
+        <mesh filename="package://mujoco_ros2_pkg/meshes/low_poly/dofbot/visual/arm_link5_low_poly.stl"/>
       </geometry>
       <material name="eerie_black"/>
@@ -174,5 +174,5 @@
       <origin rpy="0 0 0" xyz="0 0 0"/>
       <geometry>
-        <mesh filename="package://dofbot_description/meshes/low_poly/dofbot/visual/arm_link5_low_poly.stl"/>
+        <mesh filename="package://mujoco_ros2_pkg/meshes/low_poly/dofbot/visual/arm_link5_low_poly.stl"/>
       </geometry>
     </collision>
@@ -197,5 +197,5 @@
       <origin rpy="0 0 0" xyz="0 0 0"/>
       <geometry>
-        <mesh filename="package://dofbot_description/meshes/low_poly/dofbot/visual/rgrip_finger1_low_poly.stl"/>
+        <mesh filename="package://mujoco_ros2_pkg/meshes/low_poly/dofbot/visual/rgrip_finger1_low_poly.stl"/>
       </geometry>
       <material name="yinmn_blue"/>
@@ -204,5 +204,5 @@
       <origin rpy="0 0 0" xyz="0 0 0"/>
       <geometry>
-        <mesh filename="package://dofbot_description/meshes/low_poly/dofbot/visual/rgrip_finger1_low_poly.stl"/>
+        <mesh filename="package://mujoco_ros2_pkg/meshes/low_poly/dofbot/visual/rgrip_finger1_low_poly.stl"/>
       </geometry>
     </collision>
@@ -227,5 +227,5 @@
       <origin rpy="0 0 0" xyz="0 0 0"/>
       <geometry>
-        <mesh filename="package://dofbot_description/meshes/low_poly/dofbot/visual/rgrip_finger2_low_poly.stl"/>
+        <mesh filename="package://mujoco_ros2_pkg/meshes/low_poly/dofbot/visual/rgrip_finger2_low_poly.stl"/>
       </geometry>
       <material name="oxford_blue"/>
@@ -234,5 +234,5 @@
       <origin rpy="0 0 0" xyz="0 0 0"/>
       <geometry>
-        <mesh filename="package://dofbot_description/meshes/low_poly/dofbot/visual/rgrip_finger2_low_poly.stl"/>
+        <mesh filename="package://mujoco_ros2_pkg/meshes/low_poly/dofbot/visual/rgrip_finger2_low_poly.stl"/>
       </geometry>
     </collision>
@@ -257,5 +257,5 @@
       <origin rpy="0 0 0" xyz="0 0 0"/>
       <geometry>
-        <mesh filename="package://dofbot_description/meshes/low_poly/dofbot/visual/rgrip_finger3_low_poly.stl"/>
+        <mesh filename="package://mujoco_ros2_pkg/meshes/low_poly/dofbot/visual/rgrip_finger3_low_poly.stl"/>
       </geometry>
       <material name="silver_lake_blue"/>
@@ -264,5 +264,5 @@
       <origin rpy="0 0 0" xyz="0 0 0"/>
       <geometry>
-        <mesh filename="package://dofbot_description/meshes/low_poly/dofbot/visual/rgrip_finger3_low_poly.stl"/>
+        <mesh filename="package://mujoco_ros2_pkg/meshes/low_poly/dofbot/visual/rgrip_finger3_low_poly.stl"/>
       </geometry>
     </collision>
@@ -287,5 +287,5 @@
       <origin rpy="0 0 0" xyz="0 0 0"/>
       <geometry>
-        <mesh filename="package://dofbot_description/meshes/low_poly/dofbot/visual/lgrip_finger1_low_poly.stl"/>
+        <mesh filename="package://mujoco_ros2_pkg/meshes/low_poly/dofbot/visual/lgrip_finger1_low_poly.stl"/>
       </geometry>
       <material name="yinmn_blue"/>
@@ -294,5 +294,5 @@
       <origin rpy="0 0 0" xyz="0 0 0"/>
       <geometry>
-        <mesh filename="package://dofbot_description/meshes/low_poly/dofbot/visual/lgrip_finger1_low_poly.stl"/>
+        <mesh filename="package://mujoco_ros2_pkg/meshes/low_poly/dofbot/visual/lgrip_finger1_low_poly.stl"/>
       </geometry>
     </collision>
@@ -317,5 +317,5 @@
       <origin rpy="0 0 0" xyz="0 0 0"/>
       <geometry>
-        <mesh filename="package://dofbot_description/meshes/low_poly/dofbot/visual/lgrip_finger2_low_poly.stl"/>
+        <mesh filename="package://mujoco_ros2_pkg/meshes/low_poly/dofbot/visual/lgrip_finger2_low_poly.stl"/>
       </geometry>
       <material name="oxford_blue"/>
@@ -324,5 +324,5 @@
       <origin rpy="0 0 0" xyz="0 0 0"/>
       <geometry>
-        <mesh filename="package://dofbot_description/meshes/low_poly/dofbot/visual/lgrip_finger2_low_poly.stl"/>
+        <mesh filename="package://mujoco_ros2_pkg/meshes/low_poly/dofbot/visual/lgrip_finger2_low_poly.stl"/>
       </geometry>
     </collision>
@@ -347,5 +347,5 @@
       <origin rpy="0 0 0" xyz="0 0 0"/>
       <geometry>
-        <mesh filename="package://dofbot_description/meshes/low_poly/dofbot/visual/lgrip_finger3_low_poly.stl"/>
+        <mesh filename="package://mujoco_ros2_pkg/meshes/low_poly/dofbot/visual/lgrip_finger3_low_poly.stl"/>
       </geometry>
       <material name="silver_lake_blue"/>
@@ -354,5 +354,5 @@
       <origin rpy="0 0 0" xyz="0 0 0"/>
       <geometry>
-        <mesh filename="package://dofbot_description/meshes/low_poly/dofbot/visual/lgrip_finger3_low_poly.stl"/>
+        <mesh filename="package://mujoco_ros2_pkg/meshes/low_poly/dofbot/visual/lgrip_finger3_low_poly.stl"/>
       </geometry>
     </collision>
@@ -367,6 +367,58 @@
     <mimic joint="grip_joint" multiplier="-1"/>
   </joint>
-  <!--<xacro:include filename="$(find ${package_name})/urdf/dofbot_gz_properties.xacro"/>
-    <xacro:include filename="$(find ${package_name})/urdf/trajectory_controller.xacro"/>-->
+  <!--<xacro:include filename="$(find ${package_name})/urdf/dofbot_gz_properties.xacro"/>-->
+  <ros2_control name="MujocoSystem" type="system">
+    <hardware>
+      <plugin>mujoco_ros2_control/MujocoSystem</plugin>
+    </hardware>
+    <joint name="arm_joint_01">
+      <command_interface name="position"/>
+      <state_interface name="position">
+        <param name="initial_value">0.0</param>
+      </state_interface>
+      <state_interface name="velocity"/>
+      <state_interface name="effort"/>
+    </joint>
+    <joint name="arm_joint_02">
+      <command_interface name="position"/>
+      <state_interface name="position">
+        <param name="initial_value">0.0</param>
+      </state_interface>
+      <state_interface name="velocity"/>
+      <state_interface name="effort"/>
+    </joint>
+    <joint name="arm_joint_03">
+      <command_interface name="position"/>
+      <state_interface name="position">
+        <param name="initial_value">0.0</param>
+      </state_interface>
+      <state_interface name="velocity"/>
+      <state_interface name="effort"/>
+    </joint>
+    <!--<joint name="arm_joint_04">
+            <command_interface name="position" />
+            <state_interface name="position">
+                <param name="initial_value">1.0</param>
+            </state_interface>
+            <state_interface name="velocity"/>
+            <state_interface name="effort"/>
+        </joint>
+        <joint name="arm_joint_05">
+            <command_interface name="position" />
+            <state_interface name="position">
+                <param name="initial_value">1.0</param>
+            </state_interface>
+            <state_interface name="velocity"/>
+            <state_interface name="effort"/>
+        </joint>-->
+    <joint name="arm_base_link">
+      <command_interface name="position"/>
+      <state_interface name="position">
+        <param name="initial_value">1.0</param>
+      </state_interface>
+      <state_interface name="velocity"/>
+      <state_interface name="effort"/>
+    </joint>
+  </ros2_control>
   <!--<xacro:include filename="$(find ${package_name})/urdf/monocular_camera_sensor.xacro"/>-->
 </robot>
